Commit message: Updated the urdf and launch file

File: robotics_packages/descriptions/arm_description/urdf/ur5e.urdf.xacro (robot description, xacro)
@@ -4,5 +4,5 @@
     <xacro:arg name="name" default="ur5e_robot"/>
     <xacro:arg name="ur_type" default="ur5e"/>
-    <xacro:arg name="tf_prefix" default=""/>
+    <xacro:arg name="tf_prefix" default="arm_"/>
     <xacro:arg name="joint_limit_params" default="$(find ur_description)/config/$(arg ur_type)/joint_limits.yaml"/>
     <xacro:arg name="kinematics_params" default="$(find ur_description)/config/$(arg ur_type)/default_kinematics.yaml"/>
@@ -13,5 +13,5 @@
     <xacro:arg name="safety_pos_margin" default="0.15"/>
     <xacro:arg name="safety_k_position" default="20"/>
-    <!-- Simulation Parameters - Define these before using -->
+    <!-- Simulation Parameters -->
     <xacro:arg name="use_fake_hardware" default="true"/>
     <xacro:arg name="fake_sensor_commands" default="false"/>
@@ -42,13 +42,19 @@
     <xacro:arg name="com_port" default="/dev/ttyUSB0"/>
     <xacro:arg name="include_ros2_control" default="true"/>
+    <!-- Mount parameters for mobile manipulation -->
+    <xacro:arg name="parent" default="arm_world"/>
+    <xacro:arg name="mount_xyz" default="0 0 0"/>
+    <xacro:arg name="mount_rpy" default="0 0 0"/>
     <!-- Include the URDF for the UR robot-->
     <xacro:include filename="$(find ur_description)/urdf/ur_macro.xacro"/>
-    <!-- Create link fixed to the world -->
-    <link name="world" />
+    <!-- I did this to only create arm_world link if using default parent -->
+    <xacro:if value="${'$(arg parent)' == 'arm_world'}">
+        <link name="arm_world" />
+    </xacro:if>
     <!-- Instantiate the UR robot macro -->
     <xacro:ur_robot
         name="$(arg name)"
         tf_prefix="$(arg tf_prefix)"
-        parent="world"
+        parent="$(arg parent)"
         joint_limits_parameters_file="$(arg joint_limit_params)"
         kinematics_parameters_file="$(arg kinematics_params)"
@@ -82,5 +88,5 @@
         script_sender_port="$(arg script_sender_port)"
         trajectory_port="$(arg trajectory_port)">
-        <origin xyz="0 0 0" rpy="0 0 0"/>
+        <origin xyz="$(arg mount_xyz)" rpy="$(arg mount_rpy)"/>
     </xacro:ur_robot>
 </robot>

File: robotics_packages/descriptions/gripper_description/urdf/gripper.urdf.xacro (robot description, xacro)
@@ -7,5 +7,5 @@
     <xacro:ur_to_robotiq
         prefix=""
-        parent="tool0"
+        parent="arm_tool0"
         child="gripper_mount_link"
         rotation="0.0"/> <!-- This is the adapter -->

File: robotics_packages/mobile_manipulation_bringup/urdf/mobile_manipulation.urdf.xacro (robot description, xacro)
@@ -1,14 +1,11 @@
 <?xml version="1.0" encoding="UTF-8"?>
 <robot name="mobile_manipulation_robot" xmlns:xacro="http://www.ros.org/wiki/xacro">
-    <!-- Arguments for configuration -->
-    <xacro:arg name="ur_type" default="ur5e"/>
-    <xacro:arg name="use_fake_hardware" default="true"/>
-    <xacro:arg name="sim_ignition" default="false"/>
-    <xacro:arg name="sim_isaac" default="false"/>
-    <xacro:arg name="com_port" default="/dev/ttyUSB0"/>
-    <xacro:arg name="tf_prefix" default=""/>
-    <!-- Include the arm-->
-    <xacro:include filename="$(find arm_description)/urdf/ur5e.urdf.xacro"/>
-    <!-- Include the gripper-->
-    <xacro:include filename="$(find gripper_description)/urdf/gripper.urdf.xacro"/>
+   <xacro:include filename="$(find husky_description)/urdf/husky.urdf.xacro"/>
+   <xacro:include filename="$(find arm_description)/urdf/ur5e.urdf.xacro"/>
+   <xacro:include filename="$(find gripper_description)/urdf/gripper.urdf.xacro"/>
+   <joint name="arm_mount_joint" type="fixed">
+       <origin xyz="0 0 0" rpy="0 0 0"/>
+       <parent link="top_plate_link"/>
+       <child link="arm_world"/>
+   </joint>
 </robot>
